File: KICAD/5-SLOT/Diego 500 5 slot.kicad_pcb (KiCad board)
At the start: 4 copper layers, 195 x 140 mm, 143 parts, among them CN1 A500 side car, CN10 1000pf, CN11 1000pf, CN12 1000pf, CN13 1000pf, CN14 1000pf, CN15 1000pf, CN16 1000pf, CN17 1000pf, CN2 Zorro 1, CN3 Zorro 2, CN4 Zorro 3, CN5 Zorro 4, CN6 Zorro 5, CN7 1000pf, CN8 1000pf, CN9 1000pf, J1 Conn_01x03_Pin, J2 A2000_CPUSLOT_EDGE_LOGICAL, J3 HDD 2, J4 HDD 1, J5 Conn_01x02_Pin, J6 ATX-24, J7 Buster, J8 Power to A500, J9 Conn_01x01_Pin, Q1 S8050, SW1 SW_Push, U1 BLUSTER, U10 74LS08, U11 501MLFT, U12 74LS32, U13 MC79M05, U2 74ALS245, U3 74LS245, U4 74LS245, U5 74LS245, U6 74LS245, U7 74ALS245, U8 74LS32, U9 MAX16054AZT_T

Commit message: Updated
Parts:
- removed D3: 1N4148, Diode_SMD:D_SOD-323
Connections:
- J6 pad 8: Net-(J6-PWR_OK) -> unconnected-(J6-PWR_OK-Pad8)
- U10 pad 1: Net-(J6-PWR_OK) -> GND
- U10 pad 2: Net-(J6-PWR_OK) -> GND
- U10 pad 3: Net-(D3-K) -> unconnected-(U10-Pad3)
Routing:
- net Net-(J6-PWR_OK): track 137.9 -> 0.00 mm, vias 1 -> 0
- net Net-(D3-K): track 3.34 -> 0.00 mm, vias 1 -> 0
- net _RST: track 202.0 -> 200.3 mm, vias 3 -> 2
