File: KICAD/5-SLOT/Diego 500 5 slot.kicad_pcb (KiCad board)
At the start: 4 copper layers, 195 x 140 mm, 142 parts, among them CN1 A500 side car, CN10 1000pf, CN11 1000pf, CN12 1000pf, CN13 1000pf, CN14 1000pf, CN15 1000pf, CN16 1000pf, CN17 1000pf, CN2 Zorro 1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

Commit message: Fix autoconfig error
Connections:
- U8 pad 10: GND -> CFG500
Routing:
- net CFG500: track 8.82 -> 26.3 mm, vias 0 -> 1
- net GND: vias 641 -> 648
Other:
- board text added: "5 slot rev 1.1"
- board text removed: "5 slot rev 1"
