File: KICAD/5-SLOT/Diego 500 5 slot.kicad_sch (KiCad schematic)
At the start: 137 parts, among them CN1 A500 side car, CN10 1000pf, CN11 1000pf, CN12 1000pf, CN13 1000pf, CN14 1000pf, CN15 1000pf, CN16 1000pf, CN17 1000pf, CN2 Zorro 1, CN3 Zorro 2, CN4 Zorro 3, CN5 Zorro 4, CN6 Zorro 5, CN7 1000pf, CN8 1000pf, CN9 1000pf, J1 Conn_01x03_Pin, J2 A2000_CPUSLOT_EDGE_LOGICAL, J3 HDD 2, J4 HDD 1, J5 Conn_01x02_Pin, J6 ATX-24, J7 Buster, J8 Power to A500, J9 Conn_01x01_Pin, Q1 S8050, SW1 SW_Push, U1 BLUSTER, U10 74LS08, U11 501MLFT, U12 74LS32, U13 MC79M05, U2 74ALS245, U3 74LS245, U4 74LS245, U5 74LS245, U6 74LS245, U7 74ALS245, U8 74LS32, U9 MAX16054AZT_T

Commit message: Updated
Parts:
- removed D3: 1N4148, Diode_SMD:D_SOD-323, symbol Device:D
- RN1, RN10, RN11, RN12, RN13, RN14, RN15, RN16, RN17, RN18, RN19, RN2, RN20, RN8, RN9: LCSC C425239 -> C20197
- RN3, RN4, RN5, RN6: LCSC C425215 -> C102665
Connections:
- net GND: now also U10.1, U10.2
- now unconnected: J6.8 (PWR_OK)
- no-connect marks 28 -> 30
Other:
- moved on the sheet: U10A

Commit message: Fix autoconfig error
Connections:
- net CFG500: now also U8.10
- net GND: no longer U8.10
Changed lines of the file:
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@@
 	(wire
 		(pts
-			(xy 93.98 40.64) (xy 97.79 40.64)
-		)
-		(stroke
-			(width 0)
-			(type default)
-		)
-	)
-	(wire
-		(pts
 			(xy 156.21 146.05) (xy 143.51 146.05)
 		)
@@
 	(wire
 		(pts
+			(xy 88.9 40.64) (xy 97.79 40.64)
+		)
+		(stroke
+			(width 0)
+			(type default)
+		)
+	)
+	(wire
+		(pts
 			(xy 527.05 318.77) (xy 534.67 318.77)
 		)
@@
 		)
 	)
+	(global_label "CFG500"
+		(shape input)
+		(at 88.9 40.64 180)
+		(fields_autoplaced yes)
+		(effects
+			(font
+				(size 1.27 1.27)
+			)
+			(justify right)
+		)
+		(property "Intersheetrefs" "${INTERSHEET_REFS}"
+			(at 78.6577 40.64 0)
+			(effects
+				(font
+					(size 1.27 1.27)
+				)
+				(justify right)
+				(hide yes)
+			)
+		)
+	)
 	(global_label "_OVR"
 		(shape output)
@@
 					(unit 1)
 				)
-			)
-		)
-	)
-	(symbol
-		(lib_id "power:GND")
-		(at 93.98 40.64 270)
-		(unit 1)
-		(exclude_from_sim no)
-		(in_bom yes)
-		(on_board yes)
-		(dnp no)
-		(property "Reference" "#PWR03"
-			(at 87.63 40.64 0)
-			(effects
-				(font
-					(size 1.27 1.27)
-				)
-				(hide yes)
-			)
-		)
-		(property "Value" "GND"
-			(at 91.186 40.64 90)
-			(effects
-				(font
-					(size 1.27 1.27)
-				)
-				(justify right)
-			)
-		)
-		(property "Footprint" ""
-			(at 93.98 40.64 0)
-			(effects
-				(font
-					(size 1.27 1.27)
-				)
-				(hide yes)
-			)
-		)
-		(property "Datasheet" ""
-			(at 93.98 40.64 0)
-			(effects
-				(font
-					(size 1.27 1.27)
-				)
-				(hide yes)
-			)
-		)
-		(property "Description" "Power symbol creates a global label with name \"GND\" , ground"
-			(at 93.98 40.64 0)
-			(effects
-				(font
-					(size 1.27 1.27)
-				)
-				(hide yes)
-			)
-		)
-		(pin "1"
-		)
-		(instances
-			(project "Zorro to 500"
-				(path "/fe999955-224f-48f7-8cb4-1836b2d4eba6"
-					(reference "#PWR03")
-					(unit 1)
-				)

Commit message: KICAD and JLC files updated
Parts:
- C23, C27, C28, C29, C31, C32: footprint Capacitor_SMD:CP_Elec_6.3x5.9 -> Capacitor_SMD:CP_Elec_6.3x7.7
- R27: value 680 -> 1k
Changed lines of the file:
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@@
 			)
 		)
-		(property "Footprint" "Capacitor_SMD:CP_Elec_6.3x5.9"
+		(property "Footprint" "Capacitor_SMD:CP_Elec_6.3x7.7"
 			(at 707.39 318.77 0)
 			(effects
@@
 			)
 		)
-		(property "Footprint" "Capacitor_SMD:CP_Elec_6.3x5.9"
+		(property "Footprint" "Capacitor_SMD:CP_Elec_6.3x7.7"
 			(at 681.99 303.53 0)
 			(effects
@@
 			)
 		)
-		(property "Footprint" "Capacitor_SMD:CP_Elec_6.3x5.9"
+		(property "Footprint" "Capacitor_SMD:CP_Elec_6.3x7.7"
 			(at 712.47 318.77 0)
 			(effects
@@
 			)
 		)
-		(property "Footprint" "Capacitor_SMD:CP_Elec_6.3x5.9"
+		(property "Footprint" "Capacitor_SMD:CP_Elec_6.3x7.7"
 			(at 731.52 331.47 0)
 			(effects
@@
 			)
 		)
-		(property "Footprint" "Capacitor_SMD:CP_Elec_6.3x5.9"
+		(property "Footprint" "Capacitor_SMD:CP_Elec_6.3x7.7"
 			(at 725.17 325.12 0)
 			(effects
@@
 			)
 		)
-		(property "Value" "680"
+		(property "Value" "1k"
 			(at 736.346 308.102 90)
 			(effects
@@
 			)
 		)
-		(property "Footprint" "Capacitor_SMD:CP_Elec_6.3x5.9"
+		(property "Footprint" "Capacitor_SMD:CP_Elec_6.3x7.7"
 			(at 718.82 318.77 0)
 			(effects
