File: KICAD/3-SLOT/Diego 500 3 slot.kicad_pcb (KiCad board)
At the start: 4 copper layers, 155 x 140 mm, 135 parts, among them CN1 A500 side car, CN10 1000pf, CN11 1000pf, CN12 1000pf, CN13 1000pf, CN14 1000pf, CN15 1000pf, CN16 1000pf, CN17 1000pf, CN2 Zorro 1, CN3 Zorro 2, CN4 Zorro 3, CN7 1000pf, CN8 1000pf, CN9 1000pf, J1 Conn_01x03_Pin, J2 A2000_CPUSLOT_EDGE_LOGICAL, J3 HDD 2, J4 HDD 1, J5 Conn_01x02_Pin, J6 ATX-24, J7 Buster, J8 Power to A500, J9 Conn_01x01_Pin, Q1 S8050, SW1 SW_Push, U1 BLUSTER, U10 74LS08, U11 501MLFT, U12 74LS32, U13 MC79M05, U2 74ALS245, U3 74LS245, U4 74LS245, U5 74LS245, U6 74LS245, U7 74ALS245, U8 74LS32, U9 MAX16054AZT_T

Commit message: General update
Routing:
- net BA10: track 110.9 -> 109.9 mm
Changed lines of the file:
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@@
 		(tags "resistor")
 		(property "Reference" "R6"
-			(at 0 1.65 360)
+			(at 0 1.65 0)
 			(layer "B.SilkS")
 			(effects
@@
 		)
 		(property "Value" "1k"
-			(at 0 -1.65 360)
+			(at 0 -1.65 0)
 			(layer "B.Fab")
 			(effects
@@
 		)
 		(fp_text user "${REFERENCE}"
-			(at 0 0 360)
+			(at 0 0 0)
 			(layer "B.Fab")
 			(effects
@@
 		(tags "resistor")
 		(property "Reference" "R22"
-			(at -3.2125 -0.2 360)
+			(at -3.2125 -0.2 0)
 			(layer "B.SilkS")
 			(effects
@@
 		)
 		(property "Value" "10k"
-			(at -3.2375 1.1 360)
+			(at -3.2375 1.1 0)
 			(layer "B.SilkS")
 			(hide yes)
@@
 		)
 		(property "LCSC" "C17414"
-			(at 0 0 360)
+			(at 0 0 0)
 			(layer "B.SilkS")
 			(hide yes)
@@
 		)
 		(fp_text user "${REFERENCE}"
-			(at 0 0 360)
+			(at 0 0 0)
 			(layer "B.Fab")
 			(effects
@@
 		(tags "resistor")
 		(property "Reference" "R20"
-			(at -0.3875 1.6 360)
+			(at -0.3875 1.6 0)
 			(layer "B.SilkS")
 			(effects
@@
 		)
 		(property "Value" "10k"
-			(at -0.4875 2.9 360)
+			(at -0.4875 2.9 0)
 			(layer "B.SilkS")
 			(effects
@@
 		)
 		(property "LCSC" "C17414"
-			(at 0 0 360)
+			(at 0 0 0)
 			(layer "B.SilkS")
 			(hide yes)
@@
 		)
 		(fp_text user "${REFERENCE}"
-			(at 0 0 360)
+			(at 0 0 0)
 			(layer "B.Fab")
 			(effects
@@
 		(tags "resistor")
 		(property "Reference" "R21"
-			(at -3.2 -0.8 360)
+			(at -3.2 -0.8 0)
 			(layer "B.SilkS")
 			(effects
@@
 		)
 		(property "Value" "10k"
-			(at -3.1 0.5 360)
+			(at -3.1 0.5 0)
 			(layer "B.SilkS")
 			(effects
@@
 		)
 		(property "LCSC" "C17414"
-			(at 0 0 360)
+			(at 0 0 0)
 			(layer "B.SilkS")
 			(hide yes)
@@
 		)
 		(fp_text user "${REFERENCE}"
-			(at 0 0 360)
+			(at 0 0 0)
 			(layer "B.Fab")
 			(effects
@@
 		(tags "resistor array")
 		(property "Reference" "RN7"
-			(at 0.2 -2.5 360)
+			(at 0.2 -2.5 0)
 			(layer "B.SilkS")
 			(effects
@@
 		(width 0.2)
 		(layer "F.Cu")
-		(net 205)
-	)
-	(segment
-		(start 106.718 253.143)
-		(end 107.663 253.143)
-		(width 0.2)
-		(layer "F.Cu")

Commit message: Fix autoconfig error
Connections:
- U8 pad 10: GND -> CFG500
Routing:
- net CFG500: track 8.82 -> 26.2 mm, vias 0 -> 1
- net Net-(J6-PS_ON#): track 129.8 -> 129.3 mm
- net +5VSB: track 107.5 -> 107.0 mm
- net GND: vias 509 -> 515
Other:
- board text added: "3 slot rev 1.1"
- board text removed: "3 slot rev 1"
