File: KICAD/3-SLOT/Diego 500 3 slot.kicad_pcb (KiCad board)
At the start: 4 copper layers, 155 x 140 mm, 135 parts, among them CN1 A500 side car, CN10 1000pf, CN11 1000pf, CN12 1000pf, CN13 1000pf, CN14 1000pf, CN15 1000pf, CN16 1000pf, CN17 1000pf, CN2 Zorro 1, CN3 Zorro 2, CN4 Zorro 3, CN7 1000pf, CN8 1000pf, CN9 1000pf, J1 Conn_01x03_Pin, J2 A2000_CPUSLOT_EDGE_LOGICAL, J3 HDD 2, J4 HDD 1, J5 Conn_01x02_Pin, J6 ATX-24, J7 Buster, J8 Power to A500, J9 Conn_01x01_Pin, Q1 S8050, SW1 SW_Push, U1 BLUSTER, U10 74LS08, U11 501MLFT, U12 74LS32, U13 MC79M05, U2 74ALS245, U3 74LS245, U4 74LS245, U5 74LS245, U6 74LS245, U7 74ALS245, U8 74LS32, U9 MAX16054AZT_T

Commit message: KICAD and JLC files updated
Parts:
- removed the G*** at (95.7, 313.6)
- added G***: LOGO, Diego Logo:Diego QR, B.Cu at (173.1, 296.0)
- C23, C27, C28, C29, C31, C32: footprint Capacitor_SMD:CP_Elec_6.3x5.9 -> Capacitor_SMD:CP_Elec_6.3x7.7
- R27: value 680 -> 1k
Routing:
- net GND: vias 515 -> 517
Other:
- board text added: "Remember to select a 7MHz clock! A500 REV3 or REV5 select CPLD A500 REV6 select A500 and close JP6 A500+ select A500 If you're using an A500 accelerator in the CO-PROCESSOR slot, you must remove the A500s CPU or E will clash! If you've got an expansion inside your A500 on the auto-config chain connect it's config out to CFGIN Only fit U11 is you need the 28mhz clock at the COPROCESSOR"
- board text removed: "Remember to select a 7MHz clock! A500 REV3 or REV5 select CPLD A500 REV6 A500 and close JP6 A500+ select A500 If you're using an A500 accelerator in the CO-PROCESSOR slot, you must remove the A500s CPU or E will clash! If you've got an expansion inside your A500 on the auto-config chain connect it's config out to CFGIN Only fit U11 is you need the 28mhz clock at the COPROCESSOR"
